File: poe.kicad_sch (KiCad schematic)
At the start: 1 part, among them U5 TPS23753APWR

Commit message: update PoE
Parts:
- added C?: 0.1uF, symbol Device:C_Small
- added C?: 1nF, symbol Device:C_Small
- added C? (x2): 1uF, symbol Device:C_Small
- added C?: 22uF, symbol Device:C_Polarized_Small
- added D?: BAV99, Package_TO_SOT_SMD:SOT-23, symbol Diode:BAV99
- added D?: D_Schottky, symbol Device:D_Schottky
- added D?: SMAJ58A, symbol Device:D_TVS
- added FB? (x2): 100, symbol Device:FerriteBead_Small
- added L?: 4.7uH, symbol Device:L_Ferrite
- added R?: 24.9k, symbol Device:R_Small
- added R?: 59k, symbol Device:R_Small
- added R? (x2): R_Small, symbol Device:R_Small
- added T?: HR051067, HR051067, symbol HR051067:HR051067
