File: MFW007B.kicad_sch (KiCad schematic)
At the start: 18 parts, among them SW1 SW_Push, SW2 SW_Push, SW3 SW_Push, SW4 SW_Push

Commit message: update 2021-03-25
Other:
- added sheet Power-over-Ethernet Conversion (poe.kicad_sch)
- sheet MCU ports: added I2C_SCL, I2C_SDA, RESET_SW, SPI_CS, SPI_IRQ, SPI_MISO, SPI_MOSI, SPI_SCK, USER_SW_1, USER_SW_2, USER_SW_3; removed none

Commit message: hook up STM32
Parts:
- added J?: Conn_01x04, symbol Connector_Generic:Conn_01x04
Connections:
- net USBDP: now reaches JIO1.A6 (DP1)
- net USBDP: now also JIO1.B6 (DP2)
- net USBDN: now reaches JIO1.A7 (DN1)
- net USBDN: now also JIO1.B7 (DN2)
- no-connect marks 7 -> 3
Other:
- removed sheet Power-over-Ethernet Conversion
- sheet MCU ports: added ETH_IRQ, I2C1_SCL, I2C1_SDA, I2C2_SCL, I2C2_SDA, SPI1_CS, SPI1_MISO, SPI1_MOSI, SPI1_SCK, SPI2_CS, SPI2_MISO, SPI2_MOSI, SPI2_SCK, USBDM, USBDP; removed I2C_SCL, I2C_SDA, SPI_CS, SPI_IRQ, SPI_MISO, SPI_MOSI, SPI_SCK

Commit message: fix some lingering issues
Connections:
- net CD: now reaches JIO2.3 (CD)
Other:
- sheet Ethernet MAC PHY ports: added ETH_CD, ETH_RDN, ETH_RDP, ETH_TDN, ETH_TDP; removed RDN, RDP, TDN, TDP
- sheet MCU ports: added RGB_LED; removed none
- company: (none) -> github.com/westrik
- title: (none) -> NA-01 Time Computer
Changed lines of the file:
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@@
 (kicad_sch (version 20201015) (generator eeschema)
   (paper "USLetter")
+  (title_block
+    (title "NA-01 Time Computer")
+    (date "2021-03-26")
+    (rev "B")
+    (company "github.com/westrik")
+    (comment 1 "MFW007")
+  )
   (junction (at 25.4 63.5) (diameter 1.016) (color 0 0 0 0))
   (junction (at 34.29 106.68) (diameter 1.016) (color 0 0 0 0))
@@
     (stroke (width 0) (type solid) (color 0 0 0 0))
   )
+  (wire (pts (xy 27.94 35.56) (xy 19.05 35.56))
+    (stroke (width 0) (type solid) (color 0 0 0 0))
+  )
   (wire (pts (xy 27.94 38.1) (xy 19.05 38.1))
     (stroke (width 0) (type solid) (color 0 0 0 0))
@@
     (stroke (width 0) (type solid) (color 0 0 0 0))
   )
+  (wire (pts (xy 88.9 88.9) (xy 99.06 88.9))
+    (stroke (width 0) (type solid) (color 0 0 0 0))
+  )
+  (wire (pts (xy 97.79 59.69) (xy 88.9 59.69))
+    (stroke (width 0) (type solid) (color 0 0 0 0))
+  )
+  (wire (pts (xy 97.79 62.23) (xy 88.9 62.23))
+    (stroke (width 0) (type solid) (color 0 0 0 0))
+  )
+  (wire (pts (xy 97.79 64.77) (xy 88.9 64.77))
+    (stroke (width 0) (type solid) (color 0 0 0 0))
+  )
+  (wire (pts (xy 97.79 67.31) (xy 88.9 67.31))
+    (stroke (width 0) (type solid) (color 0 0 0 0))
+  )
   (wire (pts (xy 99.06 30.48) (xy 109.22 30.48))
     (stroke (width 0) (type solid) (color 0 0 0 0))
   )
-  (wire (pts (xy 99.06 58.42) (xy 90.17 58.42))
-    (stroke (width 0) (type solid) (color 0 0 0 0))
-  )
-  (wire (pts (xy 99.06 60.96) (xy 90.17 60.96))
-    (stroke (width 0) (type solid) (color 0 0 0 0))
-  )
-  (wire (pts (xy 99.06 63.5) (xy 90.17 63.5))
-    (stroke (width 0) (type solid) (color 0 0 0 0))
-  )
-  (wire (pts (xy 99.06 66.04) (xy 90.17 66.04))
-    (stroke (width 0) (type solid) (color 0 0 0 0))
-  )
   (wire (pts (xy 99.06 91.44) (xy 88.9 91.44))
     (stroke (width 0) (type solid) (color 0 0 0 0))
@@
   )
   (wire (pts (xy 185.42 106.68) (xy 198.12 106.68))
+    (stroke (width 0) (type solid) (color 0 0 0 0))
+  )
+  (wire (pts (xy 185.42 113.03) (xy 198.12 113.03))
     (stroke (width 0) (type solid) (color 0 0 0 0))
   )
@@
     (effects (font (size 1.27 1.27) (thickness 0.254) bold) (justify left bottom))
   )
-  (text "TODO: hook up LEDs" (at 226.06 134.62 180)
-    (effects (font (size 1.524 1.524) (thickness 0.3048) bold italic) (justify right bottom))
-  )
   (text "Power LED" (at 232.41 124.46 0)
     (effects (font (size 1.27 1.27) (thickness 0.254) bold) (justify left bottom))
@@
     (effects (font (size 0.9906 0.9906)) (justify left bottom))
   )
+  (text "TODO: hook up LEDs" (at 246.38 118.11 180)
+    (effects (font (size 1.524 1.524) (thickness 0.3048) bold italic) (justify right bottom))
+  )
   (text "NTP LED" (at 252.73 124.46 0)
     (effects (font (size 1.27 1.27) (thickness 0.254) bold) (justify left bottom))
@@
     (effects (font (size 1.27 1.27)) (justify left bottom))
   )
+  (label "CD" (at 19.05 35.56 0)
+    (effects (font (size 1.27 1.27)) (justify left bottom))
+  )
   (label "TDN" (at 19.05 38.1 0)
     (effects (font (size 1.27 1.27)) (justify left bottom))
@@
     (effects (font (size 1.27 1.27)) (justify left bottom))
   )
+  (label "V1P" (at 88.9 59.69 0)
+    (effects (font (size 1.27 1.27)) (justify left bottom))
+  )
+  (label "V1N" (at 88.9 62.23 0)
+    (effects (font (size 1.27 1.27)) (justify left bottom))
+  )
+  (label "V2P" (at 88.9 64.77 0)
+    (effects (font (size 1.27 1.27)) (justify left bottom))
+  )
+  (label "V2N" (at 88.9 67.31 0)
+    (effects (font (size 1.27 1.27)) (justify left bottom))
+  )
   (label "TDP" (at 88.9 83.82 0)
     (effects (font (size 1.27 1.27)) (justify left bottom))
@@
     (effects (font (size 1.27 1.27)) (justify left bottom))
   )
+  (label "CD" (at 88.9 88.9 0)
+    (effects (font (size 1.27 1.27)) (justify left bottom))
+  )
   (label "RDP" (at 88.9 91.44 0)
     (effects (font (size 1.27 1.27)) (justify left bottom))
@@
     (effects (font (size 1.27 1.27)) (justify left bottom))
   )
-  (label "V1P" (at 90.17 58.42 0)
-    (effects (font (size 1.27 1.27)) (justify left bottom))
-  )
-  (label "V1N" (at 90.17 60.96 0)
-    (effects (font (size 1.27 1.27)) (justify left bottom))
-  )
-  (label "V2P" (at 90.17 63.5 0)
-    (effects (font (size 1.27 1.27)) (justify left bottom))
-  )
-  (label "V2N" (at 90.17 66.04 0)
-    (effects (font (size 1.27 1.27)) (justify left bottom))
-  )
   (label "RESET_SW" (at 109.22 30.48 180)
     (effects (font (size 1.27 1.27)) (justify right bottom))
@@
   )
   (label "USER_SW_3" (at 198.12 106.68 180)
+    (effects (font (size 1.27 1.27)) (justify right bottom))
+  )
+  (label "RGB_LED" (at 198.12 113.03 180)
     (effects (font (size 1.27 1.27)) (justify right bottom))
   )
@@
       (effects (font (size 1.27 1.27)) (justify left top))
     )
-    (pin "TDN" input (at 99.06 86.36 180)
-      (effects (font (size 1.27 1.27)) (justify left))
-    )
-    (pin "TDP" input (at 99.06 83.82 180)
-      (effects (font (size 1.27 1.27)) (justify left))
-    )
-    (pin "RDP" input (at 99.06 91.44 180)
-      (effects (font (size 1.27 1.27)) (justify left))
-    )
-    (pin "RDN" input (at 99.06 93.98 180)
-      (effects (font (size 1.27 1.27)) (justify left))
-    )
     (pin "ETHLINKLED" output (at 99.06 99.06 180)
       (effects (font (size 1.27 1.27)) (justify left))
@@
     (pin "MOSI" output (at 134.62 91.44 0)
       (effects (font (size 1.27 1.27)) (justify right))
+    )
+    (pin "ETH_RDP" input (at 99.06 91.44 180)
+      (effects (font (size 1.27 1.27)) (justify left))
+    )
+    (pin "ETH_RDN" input (at 99.06 93.98 180)
+      (effects (font (size 1.27 1.27)) (justify left))
+    )
+    (pin "ETH_TDN" input (at 99.06 86.36 180)
+      (effects (font (size 1.27 1.27)) (justify left))
+    )
+    (pin "ETH_TDP" input (at 99.06 83.82 180)
+      (effects (font (size 1.27 1.27)) (justify left))
+    )
+    (pin "ETH_CD" input (at 99.06 88.9 180)
+      (effects (font (size 1.27 1.27)) (justify left))
     )
   )
@@
       (effects (font (size 1.27 1.27)) (justify right))
     )
+    (pin "RGB_LED" output (at 185.42 113.03 0)
+      (effects (font (size 1.27 1.27)) (justify right))
+    )

Commit message: hook up mac eeprom to i2c
Connections:
- net V1N: now also J?.2 (Pin_2)
- net V1P: now also J?.1 (Pin_1)
- net V2N: now also J?.4 (Pin_4)
- net V2P: now also J?.3 (Pin_3)
Other:
- sheet Ethernet MAC PHY ports: added SCL, SDA; removed none
- moved on the sheet: J?
Changed lines of the file:
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@@
+    (stroke (width 0) (type solid) (color 0 0 0 0))
+  )
+  (wire (pts (xy 134.62 99.06) (xy 149.86 99.06))
+    (stroke (width 0) (type solid) (color 0 0 0 0))
+  )
+  (wire (pts (xy 134.62 101.6) (xy 149.86 101.6))
     (stroke (width 0) (type solid) (color 0 0 0 0))
   )
@@
     (stroke (width 0) (type solid) (color 0 0 0 0))
   )
-  (wire (pts (xy 149.86 99.06) (xy 137.16 99.06))
-    (stroke (width 0) (type solid) (color 0 0 0 0))
-  )
-  (wire (pts (xy 149.86 101.6) (xy 137.16 101.6))
-    (stroke (width 0) (type solid) (color 0 0 0 0))
-  )
   (wire (pts (xy 149.86 106.68) (xy 137.16 106.68))
     (stroke (width 0) (type solid) (color 0 0 0 0))
@@
   )
   (wire (pts (xy 208.28 157.48) (xy 200.66 157.48))
+    (stroke (width 0) (type solid) (color 0 0 0 0))
+  )
+  (wire (pts (xy 234.95 72.39) (xy 247.65 72.39))
+    (stroke (width 0) (type solid) (color 0 0 0 0))
+  )
+  (wire (pts (xy 234.95 74.93) (xy 247.65 74.93))
+    (stroke (width 0) (type solid) (color 0 0 0 0))
+  )
+  (wire (pts (xy 247.65 80.01) (xy 234.95 80.01))
+    (stroke (width 0) (type solid) (color 0 0 0 0))
+  )
+  (wire (pts (xy 247.65 82.55) (xy 234.95 82.55))
+    (stroke (width 0) (type solid) (color 0 0 0 0))
+  )
+  (wire (pts (xy 247.65 87.63) (xy 234.95 87.63))
+    (stroke (width 0) (type solid) (color 0 0 0 0))
+  )
+  (wire (pts (xy 247.65 90.17) (xy 234.95 90.17))
+    (stroke (width 0) (type solid) (color 0 0 0 0))
+  )
+  (wire (pts (xy 247.65 92.71) (xy 234.95 92.71))
+    (stroke (width 0) (type solid) (color 0 0 0 0))
+  )
+  (wire (pts (xy 247.65 95.25) (xy 234.95 95.25))
     (stroke (width 0) (type solid) (color 0 0 0 0))
   )
@@
   (label "USER_SW_3" (at 208.28 30.48 180)
     (effects (font (size 1.27 1.27)) (justify right bottom))
+  )
+  (label "I2C1_SCL" (at 234.95 72.39 0)
+    (effects (font (size 1.27 1.27)) (justify left bottom))
+  )
+  (label "I2C1_SDA" (at 234.95 74.93 0)
+    (effects (font (size 1.27 1.27)) (justify left bottom))
+  )
+  (label "I2C2_SCL" (at 234.95 80.01 0)
+    (effects (font (size 1.27 1.27)) (justify left bottom))
+  )
+  (label "I2C2_SDA" (at 234.95 82.55 0)
+    (effects (font (size 1.27 1.27)) (justify left bottom))
+  )
+  (label "SPI2_CS" (at 234.95 87.63 0)
+    (effects (font (size 1.27 1.27)) (justify left bottom))
+  )
+  (label "SPI2_SCK" (at 234.95 90.17 0)
+    (effects (font (size 1.27 1.27)) (justify left bottom))
+  )
+  (label "SPI2_MISO" (at 234.95 92.71 0)
+    (effects (font (size 1.27 1.27)) (justify left bottom))
+  )
+  (label "SPI2_MOSI" (at 234.95 95.25 0)
+    (effects (font (size 1.27 1.27)) (justify left bottom))
   )
   (symbol (lib_id "power:PWR_FLAG") (at 39.37 93.98 0) (unit 1)
@@
     )
   )
-  (symbol (lib_id "Connector_Generic:Conn_01x04") (at 124.46 60.96 0) (unit 1)
-    (in_bom yes) (on_board yes)
-    (property "Reference" "J?" (id 0) (at 126.4921 61.1314 0)
-      (effects (font (size 1.27 1.27)) (justify left))
-    )
-    (property "Value" "Conn_01x04" (id 1) (at 126.4921 63.4301 0)
-      (effects (font (size 1.27 1.27)) (justify left))
-    )
-    (property "Footprint" "" (id 2) (at 124.46 60.96 0)
-      (effects (font (size 1.27 1.27)) hide)
-    )
-    (property "Datasheet" "~" (id 3) (at 124.46 60.96 0)
+  (symbol (lib_id "Connector_Generic:Conn_01x04") (at 102.87 62.23 0) (unit 1)
+    (in_bom yes) (on_board yes)
+    (property "Reference" "J?" (id 0) (at 104.9021 62.4014 0)
+      (effects (font (size 1.27 1.27)) (justify left))
+    )
+    (property "Value" "Conn_01x04" (id 1) (at 104.9021 64.7001 0)
+      (effects (font (size 1.27 1.27)) (justify left))
+    )
+    (property "Footprint" "" (id 2) (at 102.87 62.23 0)
+      (effects (font (size 1.27 1.27)) hide)
+    )
+    (property "Datasheet" "~" (id 3) (at 102.87 62.23 0)
       (effects (font (size 1.27 1.27)) hide)
     )
@@
       (effects (font (size 1.27 1.27)) (justify left))
     )
-  )
+    (pin "SDA" input (at 134.62 101.6 0)
+      (effects (font (size 1.27 1.27)) (justify right))
+    )
+    (pin "SCL" input (at 134.62 99.06 0)
+      (effects (font (size 1.27 1.27)) (justify right))
+    )
+  )

Commit message: fix label assignments and add 2x7 header
Parts:
- removed J?: Conn_01x04, symbol Connector_Generic:Conn_01x04
- added J2: Conn_02x07, Connector_PinHeader_2.54mm:PinHeader_2x07_P2.54mm_Vertical, symbol Connector_Generic:Conn_02x07_Odd_Even
- added J3: 4P JST-SH, Connector_JST:JST_SH_SM04B-SRSS-TB_1x04-1MP_P1.00mm_Horizontal, symbol PoE-NTP-Clock-rescue:Conn_01x04-Connector_Generic
Connections:
- net +5V: now also J2.1 (Pin_1), J3.3 (Pin_3)
- net GND: now also J2.2 (Pin_2), J3.4 (Pin_4)
- net I2C1_SCL: now also J2.3 (Pin_3), J3.1 (Pin_1)
- net I2C1_SDA: now also J2.4 (Pin_4), J3.2 (Pin_2)
- net I2C2_SCL: now also J2.5 (Pin_5)
- net I2C2_SDA: now also J2.6 (Pin_6)
- net SPI2_CS: now also J2.7 (Pin_7)
- net SPI2_MISO: now also J2.9 (Pin_9)
- net SPI2_MOSI: now also J2.10 (Pin_10)
- net SPI2_SCK: now also J2.8 (Pin_8)
- net V1N: now also J2.12 (Pin_12)
- net V1P: now also J2.11 (Pin_11)
- net V2N: now also J2.14 (Pin_14)
- net V2P: now also J2.13 (Pin_13)

Commit message: rough component placement
Parts:
- added D4: B5819W, Diode_SMD:D_SOD-123, symbol Device:D_Schottky
- added R27, R28: 1K, Resistor_SMD:R_0402_1005Metric, symbol Device:R_Small
- added R29, R30, R31: 330, Resistor_SMD:R_0402_1005Metric, symbol Device:R_Small
- C1: footprint Capacitor_SMD:C_0402_1005Metric -> Capacitor_SMD:C_0805_2012Metric
- D2, D3: symbol PoE-NTP-Clock-rescue:LED-Device -> Device:LED
- H1, H2, H3, H4: symbol PoE-NTP-Clock-rescue:MountingHole-Mechanical -> Mechanical:MountingHole
- J3: symbol PoE-NTP-Clock-rescue:Conn_01x04-Connector_Generic -> Connector_Generic:Conn_01x04
- JIO2: symbol PoE-NTP-Clock-rescue:WE-RJ45_74984104400-WE-RJ45_74984104400 -> WE-RJ45_74984104400:WE-RJ45_74984104400
- JP1, JP2: symbol PoE-NTP-Clock-rescue:Jumper-Device -> Jumper:Jumper_2_Bridged
- SW1, SW2, SW3, SW4: symbol PoE-NTP-Clock-rescue:SW_Push-Switch -> Switch:SW_Push
Connections:
- net ETHLED1P is gone; now on an unnamed net: JIO2.11
- net ETHLED2P is gone; now on an unnamed net: JIO2.13
- net +5V: now also D4.1 (K); no longer JIO1.A4 (VBUS), JIO1.A9 (VBUS), JIO1.B4 (VBUS), JIO1.B9 (VBUS)
- net ETHACTLED: now also R27.2
- net ETHLINKLED: now also R28.1
- net GND: now also JP2.2 (B)
- net RGB_LED: now also R29.1; no longer D1.4 (DIN)
- net at D3.1 (K): now also R31.1
- net NTP_LED: now reaches D3.2 (A)
- net at D2.1 (K): now also R30.1
- net +3V3: now reaches D2.2 (A)
- net +3V3: now also JP1.1 (A)
- net STLEDGND: now reaches JP2.1 (A)
- net STLEDGND: now also R30.2, R31.2
- net ETHLED1N: no longer names the net of JIO2.12
- net ETHLED1N: now also R27.1
- net ETHLED2N: no longer names the net of JIO2.14
- net ETHLED2N: now also R28.2
- new net: D4.2 (A), JIO1.A4 (VBUS), JIO1.A9 (VBUS), JIO1.B4 (VBUS), JIO1.B9 (VBUS)
- new net: D1.4 (DIN), R29.2
Other:
- sheet MCU ports: added NTP_LED; removed none
- note removed: "TODO: hook up LEDs"
- moved on the sheet: D1, D2, D3, H1, H2, H3, H4, J2, J3, JP1, JP2
