File: MFW007B.kicad_sch (KiCad schematic)
At the start: 26 parts, among them J2 Conn_02x07, J3 4P JST-SH, SW1 SW_Push, SW2 SW_Push, SW3 SW_Push, SW4 SW_Push

Commit message: add some part numbers to schematic
Parts:
- C1: LCSC Part Number (none) -> C1710
- D1, H1, H2, H3, H4, J2, J3, JIO2, JP1, JP2, SW1, SW2, SW3, SW4: LCSC Part Number (none) -> N/A
- D2: LCSC Part Number (none) -> C2286
- D3: LCSC Part Number (none) -> C72043
- D4: LCSC Part Number (none) -> C8598
- JIO1: LCSC Part Number (none) -> N/A; LED (none) -> WE-RJ45_74984104400; MANUFACTURER Global Connector Technology -> WE-RJ45_74984104400:74984104400; MAXIMUM_PACKAGE_HEIGHT 3.46mm -> (none); MOUNT (none) -> 10/100 Base-T; MPN (none) -> https://www.we-online.com/catalog/datasheet/74984104400.pdf; Manufacturer (none) -> N/A; Manufacturer Part Number (none) -> green/yellow-green/yellow; PARTREV A2 -> (none); POE (none) -> THR; STANDARD Manufacturer Recommendations -> (none); VALUE (none) -> 74984104400
- R1, R2: LCSC Part Number (none) -> C25905
Changed lines of the file:
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@@
+      (effects (font (size 1.27 1.27)) hide)
+    )
+    (property "LCSC Part Number" "C25905" (id 4) (at 38.1 99.06 0)
       (effects (font (size 1.27 1.27)) hide)
     )
@@
       (effects (font (size 1.27 1.27)) hide)
     )
+    (property "LCSC Part Number" "C25905" (id 4) (at 38.1 101.6 0)
+      (effects (font (size 1.27 1.27)) hide)
+    )
   )
   (symbol (lib_id "Device:R_Small") (at 63.5 43.18 90) (unit 1)
@@
       (effects (font (size 1.27 1.27)) hide)
     )
+    (property "LCSC Part Number" "N/A" (id 4) (at 237.49 149.86 0)
+      (effects (font (size 1.27 1.27)) hide)
+    )
   )
   (symbol (lib_id "Mechanical:MountingHole") (at 237.49 154.94 0) (unit 1)
@@
       (effects (font (size 1.27 1.27)) hide)
     )
+    (property "LCSC Part Number" "N/A" (id 4) (at 237.49 154.94 0)
+      (effects (font (size 1.27 1.27)) hide)
+    )
   )
   (symbol (lib_id "Mechanical:MountingHole") (at 237.49 160.02 0) (unit 1)
@@
       (effects (font (size 1.27 1.27)) hide)
     )
+    (property "LCSC Part Number" "N/A" (id 4) (at 237.49 160.02 0)
+      (effects (font (size 1.27 1.27)) hide)
+    )
   )
   (symbol (lib_id "Mechanical:MountingHole") (at 237.49 165.1 0) (unit 1)
@@
       (effects (font (size 1.27 1.27)) hide)
     )
+    (property "LCSC Part Number" "N/A" (id 4) (at 237.49 165.1 0)
+      (effects (font (size 1.27 1.27)) hide)
+    )
   )
   (symbol (lib_id "Device:C_Small") (at 58.42 114.3 0) (unit 1)
@@
     )
     (property "Datasheet" "~" (id 3) (at 58.42 114.3 0)
+      (effects (font (size 1.27 1.27)) hide)
+    )
+    (property "LCSC Part Number" "C1710" (id 4) (at 58.42 114.3 0)
       (effects (font (size 1.27 1.27)) hide)
     )
@@
       (effects (font (size 1.27 1.27)) hide)
     )
+    (property "LCSC Part Number" "C8598" (id 4) (at 45.72 93.98 0)
+      (effects (font (size 1.27 1.27)) hide)
+    )
   )
   (symbol (lib_id "Jumper:Jumper_2_Bridged") (at 58.42 31.75 270) (unit 1)
@@
     )
     (property "Datasheet" "~" (id 3) (at 58.42 31.75 0)
+      (effects (font (size 1.27 1.27)) hide)
+    )
+    (property "LCSC Part Number" "N/A" (id 4) (at 58.42 31.75 0)
       (effects (font (size 1.27 1.27)) hide)
     )
@@
       (effects (font (size 1.27 1.27)) hide)
     )
+    (property "LCSC Part Number" "N/A" (id 4) (at 245.11 90.17 0)
+      (effects (font (size 1.27 1.27)) hide)
+    )
   )
   (symbol (lib_id "Device:LED") (at 232.41 57.15 90) (unit 1)
@@
       (effects (font (size 1.27 1.27)) hide)
     )
+    (property "LCSC Part Number" "C2286" (id 4) (at 232.41 57.15 0)
+      (effects (font (size 1.27 1.27)) hide)
+    )
   )
   (symbol (lib_id "Device:LED") (at 252.73 57.15 90) (unit 1)
@@
     )
     (property "Datasheet" "~" (id 3) (at 252.73 57.15 0)
+      (effects (font (size 1.27 1.27)) hide)
+    )
+    (property "LCSC Part Number" "C72043" (id 4) (at 252.73 57.15 0)
       (effects (font (size 1.27 1.27)) hide)
     )
@@
       (effects (font (size 1.27 1.27)) hide)
     )
+    (property "LCSC Part Number" "N/A" (id 4) (at 93.98 30.48 0)
+      (effects (font (size 1.27 1.27)) hide)
+    )
   )
   (symbol (lib_id "Switch:SW_Push") (at 134.62 30.48 0) (unit 1)
@@
       (effects (font (size 1.27 1.27)) hide)
     )
+    (property "LCSC Part Number" "N/A" (id 4) (at 134.62 30.48 0)
+      (effects (font (size 1.27 1.27)) hide)
+    )
   )
   (symbol (lib_id "Switch:SW_Push") (at 162.56 30.48 0) (unit 1)
@@
       (effects (font (size 1.27 1.27)) hide)
     )
+    (property "LCSC Part Number" "N/A" (id 4) (at 162.56 30.48 0)
+      (effects (font (size 1.27 1.27)) hide)
+    )
   )
   (symbol (lib_id "Switch:SW_Push") (at 193.04 30.48 0) (unit 1)
@@
       (effects (font (size 1.27 1.27)) hide)
     )
+    (property "LCSC Part Number" "N/A" (id 4) (at 193.04 30.48 0)
+      (effects (font (size 1.27 1.27)) hide)
+    )
   )
   (symbol (lib_id "Connector_Generic:Conn_01x04") (at 35.56 162.56 0) (unit 1)
@@
     )
     (property "Datasheet" "~" (id 3) (at 35.56 162.56 0)
+      (effects (font (size 1.27 1.27)) hide)
+    )
+    (property "LCSC Part Number" "N/A" (id 4) (at 35.56 162.56 0)
       (effects (font (size 1.27 1.27)) hide)
     )
@@
       (effects (font (size 1.27 1.27)) hide)
     )
+    (property "LCSC Part Number" "N/A" (id 4) (at 34.29 191.77 0)
+      (effects (font (size 1.27 1.27)) hide)
+    )
   )
   (symbol (lib_id "LED:WS2812B") (at 242.57 30.48 0) (unit 1)
@@
     (property "Datasheet" "https://cdn-shop.adafruit.com/datasheets/WS2812B.pdf" (id 3) (at 245.11 40.005 0)
       (effects (font (size 1.27 1.27)) (justify left top) hide)
+    )
+    (property "LCSC Part Number" "N/A" (id 4) (at 242.57 30.48 0)
+      (effects (font (size 1.27 1.27)) hide)
     )
   )
@@
       (effects (font (size 1.27 1.27)) (justify left bottom) hide)
     )
-    (property "MAXIMUM_PACKAGE_HEIGHT" "3.46mm" (id 4) (at 25.4 109.22 0)
-      (effects (font (size 1.27 1.27)) (justify left bottom) hide)
-    )
-    (property "PARTREV" "A2" (id 5) (at 25.4 109.22 0)
-      (effects (font (size 1.27 1.27)) (justify left bottom) hide)
-    )
-    (property "STANDARD" "Manufacturer Recommendations" (id 6) (at 25.4 109.22 0)
-      (effects (font (size 1.27 1.27)) (justify left bottom) hide)
-    )
-    (property "MANUFACTURER" "Global Connector Technology" (id 7) (at 25.4 109.22 0)
-      (effects (font (size 1.27 1.27)) (justify left bottom) hide)
+    (property "MAXIMUM_PACKAGE_HEIGHT" "" (id 4) (at 25.4 109.22 0)
+      (effects (font (size 1.27 1.27)) (justify left bottom) hide)
+    )
+    (property "PARTREV" "" (id 5) (at 25.4 109.22 0)
+      (effects (font (size 1.27 1.27)) (justify left bottom) hide)
+    )
+    (property "STANDARD" "" (id 6) (at 25.4 109.22 0)
+      (effects (font (size 1.27 1.27)) (justify left bottom) hide)
+    )
+    (property "MANUFACTURER" "WE-RJ45_74984104400:74984104400" (id 7) (at 25.4 109.22 0)
+      (effects (font (size 1.27 1.27)) (justify left bottom) hide)
+    )
+    (property "LCSC Part Number" "N/A" (id 4) (at 25.4 109.22 0)
+      (effects (font (size 1.27 1.27)) hide)
+    )
+    (property "LED" "WE-RJ45_74984104400" (id 5) (at 25.4 109.22 0)
+      (effects (font (size 1.27 1.27)) hide)
+    )
+    (property "MOUNT" "10/100 Base-T" (id 6) (at 25.4 109.22 0)
+      (effects (font (size 1.27 1.27)) hide)
+    )
+    (property "MPN" "https://www.we-online.com/catalog/datasheet/74984104400.pdf" (id 7) (at 25.4 109.22 0)
+      (effects (font (size 1.27 1.27)) hide)
+    )
+    (property "Manufacturer" "N/A" (id 8) (at 25.4 109.22 0)
+      (effects (font (size 1.27 1.27)) hide)
+    )
+    (property "Manufacturer Part Number" "green/yellow-green/yellow" (id 9) (at 25.4 109.22 0)
+      (effects (font (size 1.27 1.27)) hide)
+    )
+    (property "POE" "THR" (id 10) (at 25.4 109.22 0)
+      (effects (font (size 1.27 1.27)) hide)
+    )
+    (property "VALUE" "74984104400" (id 11) (at 25.4 109.22 0)
+      (effects (font (size 1.27 1.27)) hide)
     )
   )
@@
       (effects (font (size 1.27 1.27)) (justify left bottom) hide)
     )
-  )
+    (property "LCSC Part Number" "N/A" (id 4) (at 40.64 45.72 0)
+      (effects (font (size 1.27 1.27)) hide)
+    )
+  )
